File: 2nd-mainboard-pcb/2nd-mainboard-pcb.kicad_pcb (KiCad board)
At the start: 4 copper layers, 99 x 97.5 mm, 132 parts, among them J1 PJ-082BH, J10 Servo Motor BL Touch, J11 T3, J12 Steckverbinder_Male_Fans, J13 Steckverbinder_Female_Leistung, J14 FAN3, J15 Steckverbinder_Female_Motoren, J16 ISP, J19 T2, J2 Fan_12/5V_Regelung, J20 T2, J21 T2, J22 T3, J23 Conn_01x04_Socket, J24 Steckverbinder_Male_Leistung, J3 Fan_12/5V_Regelung, J4 FAN0, J5 FAN1, J6 FAN2, J7 Stepper Motor, J8 Servo Motor SM, J9 Microstepping, P1 USB_C_Receptacle_USB2.0_14P, SW3 PTS820 J25K SMTR LFS, U1 SQJ409EP-T1_GE3, U10 ATmega328PB-A, U12 MPU-6050, U2 SZ1SMB5927BT3G, U4 TPS565208, U5 FT232RL, U6 TPS56837RPAR, U7 TPM16050-S6TR, U8 RJK0456DPB-00-J5, U9 RJK0456DPB-00-J5, Y1 ECS-160-18-4X-CKM

Commit message: no more errors
Parts:
- moved U1 1.28 mm to (133.8, 127.7), turned to 0 degrees
- turned U2 to -90 degrees
Routing:
- net GND: track 307.1 -> 317.5 mm
- net RESET: track 113.1 -> 109.7 mm
- net PWR_IN_PROT: track 15.3 -> 13.0 mm
- net Net-(D7-K): track 0.00 -> 1.99 mm
- net Net-(U1-G): track 23.7 -> 24.3 mm
- added copper zone on F.Cu, net AREF
- added copper zone on B.Cu, net GND
